File: KiCAD/MCU-Link_MR/mculink_kicad_power_usb.kicad_sch (KiCad schematic)
At the start: 39 parts, among them J9 USB4110-GF-A_REVB, U1 LPC55S69JBD64, U2 XC6227C331PR-G, Y1 NX3225GB-16M-STD-CRA-2

Commit message: updated BOM with new part numbers
Parts:
- C1: value 4.7uF 6.3V -> 4.7uF 25V; mouser# 581-06033D475KAT2A -> 581-CM05X5R475M25AH
- C10, C26, C7, C8, C9: value 10nF 6.3V -> 10nF 25V; mouser# 80-C0603C103M5R -> 81-GXT155R71E103KE1D
- C11, C12: value 8pF 6.3V -> 8pF 50V; mouser# 810-C1608C0G1H080D -> 81-GJM1555C1H8R0DB1D
- C13, C17, C2, C20, C23, C24, C3, C4, C5, C6: value 100nF 6.3V -> 100nF 25V; mouser# 80-C0603C104K9R -> 963-MLAST105SB5104KF
- C14, C16, C21: value 47pF 6.3V -> 47pF 50V; mouser# 80-C0603C470M5HACTU -> 77-VJ0402A470FXACBC
- C15, C18, C19: value 22uF 6.3V -> 22uF 10V; mouser# 581-KGM15CR50J226MT -> 81-GRM158R61A226ME5D
- C22, C25: value 10uF 6.3V -> 10uF 10V; mouser# 581-06036D106MAT2A -> 81-GRT155R61A16ME13J
- R1: value 10k 5% 100mW -> 10k 1% 63mW; mouser# 667-ERJ-3GEYJ103V -> 71-CRCW040210K0FKEDC
- R2: value 20k 5% 100mW -> 20k 5% 63mW; mouser# 652-CR0603JW-203ELF -> 71-CRCW040220K0JNEDC
- R4, R7: value 5.1k 5% 100mW -> 5.1k 5% 63mW; mouser# 652-CR0603JW-512ELF -> 71-CRCW04025K10JNEDC
Changed lines of the file:
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@@
 			)
 		)
-		(property "Value" "100nF 6.3V"
+		(property "Value" "100nF 25V"
 			(at 261.874 101.092 90)
 			(effects
@@
 			)
 		)
-		(property "mouser#" "80-C0603C104K9R"
+		(property "mouser#" "963-MLAST105SB5104KF"
 			(at 257.81 88.9 0)
 			(effects
@@
 			)
 		)
-		(property "Value" "47pF 6.3V"
+		(property "Value" "47pF 50V"
 			(at 250.19 99.314 90)
 			(effects
@@
 			)
 		)
-		(property "mouser#" "80-C0603C470M5HACTU"
+		(property "mouser#" "77-VJ0402A470FXACBC"
 			(at 246.38 88.9 0)
 			(effects
@@
 			)
 		)
-		(property "Value" "22uF 6.3V"
+		(property "Value" "22uF 10V"
 			(at 239.522 99.822 90)
 			(effects
@@
 			)
 		)
-		(property "mouser#" "581-KGM15CR50J226MT"
+		(property "mouser#" "81-GRM158R61A226ME5D"
 			(at 234.95 88.9 0)
 			(effects
@@
 			)
 		)
-		(property "Value" "22uF 6.3V"
+		(property "Value" "22uF 10V"
 			(at 273.558 99.568 90)
 			(effects
@@
 			)
 		)
-		(property "mouser#" "581-KGM15CR50J226MT"
+		(property "mouser#" "81-GRM158R61A226ME5D"
 			(at 269.24 88.9 0)
 			(effects
@@
 			)
 		)
-		(property "Value" "8pF 6.3V"
+		(property "Value" "8pF 50V"
 			(at 233.172 61.214 90)
 			(effects
@@
 			)
 		)
-		(property "mouser#" "810-C1608C0G1H080D"
+		(property "mouser#" "81-GJM1555C1H8R0DB1D"
 			(at 228.6 52.07 0)
 			(effects
@@
 			)
 		)
-		(property "Value" "8pF 6.3V"
+		(property "Value" "8pF 50V"
 			(at 259.08 60.96 90)
 			(effects
@@
 			)
 		)
-		(property "mouser#" "810-C1608C0G1H080D"
+		(property "mouser#" "81-GJM1555C1H8R0DB1D"
 			(at 254 52.07 0)
 			(effects
@@
 			)
 		)
-		(property "Value" "10nF 6.3V"
+		(property "Value" "10nF 25V"
 			(at 101.981 140.843 0)
 			(effects
@@
 			)
 		)
-		(property "mouser#" "80-C0603C103M5R"
+		(property "mouser#" "81-GXT155R71E103KE1D"
 			(at 99.06 139.7 0)
 			(effects
@@
 			)
 		)
-		(property "Value" "10k 5% 100mW"
+		(property "Value" "10k 1% 63mW"
 			(at 116.84 111.3536 90)
 			(effects
@@
 			)
 		)
-		(property "mouser#" "667-ERJ-3GEYJ103V"
+		(property "mouser#" "71-CRCW040210K0FKEDC"
 			(at 116.84 114.3 0)
 			(effects
@@
 			)
 		)
-		(property "Value" "20k 5% 100mW"
+		(property "Value" "20k 5% 63mW"
 			(at 124.968 123.063 0)
 			(effects
@@
 			)
 		)
-		(property "mouser#" "652-CR0603JW-203ELF"
+		(property "mouser#" "71-CRCW040220K0JNEDC"
 			(at 123.19 121.92 0)
 			(effects
@@
 			)
 		)
-		(property "Value" "100nF 6.3V"
+		(property "Value" "100nF 25V"
 			(at 41.402 103.886 90)
 			(effects
@@
 			)
 		)
-		(property "mouser#" "80-C0603C104K9R"
+		(property "mouser#" "963-MLAST105SB5104KF"
 			(at 36.83 92.71 0)
 			(effects
@@
 			)
 		)
-		(property "Value" "10uF 6.3V"
+		(property "Value" "10uF 10V"
 			(at 28.956 103.378 90)
 			(effects
@@
 			)
 		)
-		(property "mouser#" "581-06036D106MAT2A"
+		(property "mouser#" "81-GRT155R61A16ME13J"
 			(at 24.13 92.71 0)
 			(effects
@@
 			)
 		)
-		(property "Value" "100nF 6.3V"
+		(property "Value" "100nF 25V"
 			(at 89.408 105.41 90)
 			(effects
@@
 			)
 		)
-		(property "mouser#" "80-C0603C104K9R"
+		(property "mouser#" "963-MLAST105SB5104KF"
 			(at 85.09 92.71 0)
 			(effects
@@
 			)
 		)
-		(property "Value" "10uF 6.3V"
+		(property "Value" "10uF 10V"
 			(at 102.108 103.124 90)
 			(effects
@@
 			)
 		)
-		(property "mouser#" "581-06036D106MAT2A"
+		(property "mouser#" "81-GRT155R61A16ME13J"
 			(at 97.79 92.71 0)
 			(effects
@@
 			)
 		)
-		(property "Value" "4.7uF 6.3V"
+		(property "Value" "4.7uF 25V"
 			(at 55.372 53.594 90)
 			(effects
@@
 			)
 		)
-		(property "mouser#" "581-06033D475KAT2A"
+		(property "mouser#" "581-CM05X5R475M25AH"
 			(at 50.8 41.91 0)
 			(effects
@@
 			)
 		)
-		(property "Value" "100nF 6.3V"
+		(property "Value" "100nF 25V"
 			(at 66.548 53.594 90)
 			(effects
@@
 			)
 		)
-		(property "mouser#" "80-C0603C104K9R"
+		(property "mouser#" "963-MLAST105SB5104KF"
 			(at 62.23 41.91 0)
 			(effects
@@
 			)
 		)
-		(property "Value" "100nF 6.3V"
+		(property "Value" "100nF 25V"
 			(at 77.216 53.34 90)
 			(effects
@@
 			)
 		)
-		(property "mouser#" "80-C0603C104K9R"
+		(property "mouser#" "963-MLAST105SB5104KF"
 			(at 73.66 41.91 0)
 			(effects
@@
 			)
 		)
-		(property "Value" "100nF 6.3V"
+		(property "Value" "100nF 25V"
 			(at 89.408 53.594 90)
 			(effects
@@
 			)
 		)
-		(property "mouser#" "80-C0603C104K9R"
+		(property "mouser#" "963-MLAST105SB5104KF"
 			(at 85.09 41.91 0)
 			(effects
@@
 			)
 		)
-		(property "Value" "100nF 6.3V"
+		(property "Value" "100nF 25V"
 			(at 101.092 53.086 90)
 			(effects
@@
 			)
 		)
-		(property "mouser#" "80-C0603C104K9R"
+		(property "mouser#" "963-MLAST105SB5104KF"
 			(at 96.52 41.91 0)
 			(effects
@@
 			)
 		)
-		(property "Value" "100nF 6.3V"
+		(property "Value" "100nF 25V"
 			(at 112.268 53.594 90)
 			(effects
@@
 			)
 		)
-		(property "mouser#" "80-C0603C104K9R"
+		(property "mouser#" "963-MLAST105SB5104KF"
 			(at 107.95 41.91 0)
 			(effects
@@
 			)
 		)
-		(property "Value" "10nF 6.3V"
+		(property "Value" "10nF 25V"
 			(at 123.698 52.832 90)
 			(effects
@@
 			)
 		)
-		(property "mouser#" "80-C0603C103M5R"
+		(property "mouser#" "81-GXT155R71E103KE1D"
 			(at 119.38 41.91 0)
 			(effects
@@
 			)
 		)
-		(property "Value" "10nF 6.3V"
+		(property "Value" "10nF 25V"
 			(at 133.858 51.816 90)
 			(effects
@@
 			)
 		)
-		(property "mouser#" "80-C0603C103M5R"
+		(property "mouser#" "81-GXT155R71E103KE1D"
 			(at 129.54 41.91 0)
 			(effects
@@
 			)
 		)
-		(property "Value" "10nF 6.3V"
+		(property "Value" "10nF 25V"
 			(at 145.288 52.07 90)
 			(effects
@@
 			)
 		)
-		(property "mouser#" "80-C0603C103M5R"
+		(property "mouser#" "81-GXT155R71E103KE1D"
 			(at 140.97 41.91 0)
 			(effects
@@
 			)
 		)
-		(property "Value" "10nF 6.3V"
+		(property "Value" "10nF 25V"
 			(at 156.718 52.07 90)
 			(effects
@@
 			)
 		)
-		(property "mouser#" "80-C0603C103M5R"
+		(property "mouser#" "81-GXT155R71E103KE1D"
 			(at 152.4 41.91 0)
 			(effects
@@
 			)
 		)
-		(property "Value" "100nF 6.3V"
+		(property "Value" "100nF 25V"
 			(at 156.464 76.962 90)
 			(effects
@@
 			)
 		)
-		(property "mouser#" "80-C0603C104K9R"
+		(property "mouser#" "963-MLAST105SB5104KF"
 			(at 152.4 64.77 0)
 			(effects
@@
 			)
 		)
-		(property "Value" "47pF 6.3V"
+		(property "Value" "47pF 50V"
 			(at 168.402 77.216 90)
 			(effects
@@
 			)
 		)
-		(property "mouser#" "80-C0603C470M5HACTU"
+		(property "mouser#" "77-VJ0402A470FXACBC"
 			(at 163.83 64.77 0)
 			(effects
@@
 			)
 		)
-		(property "Value" "100nF 6.3V"
+		(property "Value" "100nF 25V"
 			(at 156.21 104.394 90)
 			(effects
@@
 			)
 		)
-		(property "mouser#" "80-C0603C104K9R"
+		(property "mouser#" "963-MLAST105SB5104KF"
 			(at 152.4 92.71 0)
 			(effects
@@
 			)
 		)
-		(property "Value" "47pF 6.3V"
+		(property "Value" "47pF 50V"
 			(at 167.64 103.632 90)
 			(effects
@@
 			)
 		)
-		(property "mouser#" "80-C0603C470M5HACTU"
+		(property "mouser#" "77-VJ0402A470FXACBC"
 			(at 163.83 92.71 0)
 			(effects
@@
 			)
 		)
-		(property "Value" "22uF 6.3V"
+		(property "Value" "22uF 10V"
 			(at 145.034 103.632 90)
 			(effects
@@
 			)
 		)
-		(property "mouser#" "581-KGM15CR50J226MT"
+		(property "mouser#" "81-GRM158R61A226ME5D"
 			(at 140.97 92.71 0)
 			(effects
@@
 			)
 		)
-		(property "Value" "5.1k 5% 100mW"
+		(property "Value" "5.1k 5% 63mW"
 			(at 49.53 188.722 90)
 			(effects
@@
 			)
 		)
-		(property "mouser#" "652-CR0603JW-512ELF"
+		(property "mouser#" "71-CRCW04025K10JNEDC"
 			(at 53.34 172.72 0)
 			(effects
@@
 			)
 		)
-		(property "Value" "5.1k 5% 100mW"
+		(property "Value" "5.1k 5% 63mW"
 			(at 60.706 189.23 90)
 			(effects
@@
 			)
 		)
-		(property "mouser#" "652-CR0603JW-512ELF"
+		(property "mouser#" "71-CRCW04025K10JNEDC"
 			(at 57.15 172.72 0)
 			(effects
