File: KiCAD/MCU-Link_MR/mculink_kicad_uart.kicad_sch (KiCad schematic)
At the start: 20 parts, among them J11 JST-GH BM06B-GHS, U10 74LVC1T45GW, U11 74LVC1T45GW, U8 74LVC1T45GW, U9 74LVC1T45GW

Commit message: finalized v0.5 for production
Parts:
- added JP2: RTS, Jumper:SolderJumper-2_P1.3mm_Bridged_RoundedPad1.0x1.5mm, symbol Jumper:SolderJumper_2_Bridged
- added JP3: CTS, Jumper:SolderJumper-2_P1.3mm_Bridged_RoundedPad1.0x1.5mm, symbol Jumper:SolderJumper_2_Bridged
Connections:
- net at D4.4 (K3), J11.4 (Pin_4): now also JP3.2 (B); no longer R6.2
- net at D4.5 (K4), D4.6 (K5), J11.5 (Pin_5): now also JP2.2 (B); no longer R25.2
- new net: JP2.1 (A), R25.2
- new net: JP3.1 (A), R6.2
Changed lines of the file:
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@@
 	(wire
 		(pts
-			(xy 97.79 55.88) (xy 97.79 173.99)
+			(xy 97.79 55.88) (xy 97.79 109.22)
 		)
 		(stroke
@@
 	(wire
 		(pts
-			(xy 95.25 53.34) (xy 95.25 129.54)
+			(xy 95.25 53.34) (xy 95.25 109.22)
 		)
 		(stroke
@@
 	(wire
 		(pts
+			(xy 97.79 116.84) (xy 97.79 173.99)
+		)
+		(stroke
+			(width 0)
+			(type default)
+		)
+	)
+	(wire
+		(pts
 			(xy 50.8 163.83) (xy 50.8 160.02)
 		)
@@
 	(wire
 		(pts
+			(xy 95.25 116.84) (xy 95.25 129.54)
+		)
+		(stroke
+			(width 0)
+			(type default)
+		)
+	)
+	(wire
+		(pts
 			(xy 50.8 115.57) (xy 52.07 115.57)
 		)
@@
 	)
 	(symbol
+		(lib_id "Jumper:SolderJumper_2_Bridged")
+		(at 97.79 113.03 90)
+		(unit 1)
+		(exclude_from_sim no)
+		(in_bom no)
+		(on_board yes)
+		(dnp no)
+		(property "Reference" "JP2"
+			(at 101.092 111.252 90)
+			(effects
+				(font
+					(size 1.27 1.27)
+				)
+			)
+		)
+		(property "Value" "RTS"
+			(at 101.346 113.284 90)
+			(effects
+				(font
+					(size 1.27 1.27)
+				)
+			)
+		)
+		(property "Footprint" "Jumper:SolderJumper-2_P1.3mm_Bridged_RoundedPad1.0x1.5mm"
+			(at 97.79 113.03 0)
+			(effects
+				(font
+					(size 1.27 1.27)
+				)
+				(hide yes)
+			)
+		)
+		(property "Datasheet" "~"
+			(at 97.79 113.03 0)
+			(effects
+				(font
+					(size 1.27 1.27)
+				)
+				(hide yes)
+			)
+		)
+		(property "Description" "Solder Jumper, 2-pole, closed/bridged"
+			(at 97.79 113.03 0)
+			(effects
+				(font
+					(size 1.27 1.27)
+				)
+				(hide yes)
+			)
+		)
+		(pin "2"
+		)
+		(pin "1"
+		)
+		(instances
+			(project ""
+				(path "/5d025764-753a-4b80-8d3d-c9a8a22c9527/00000000-0000-0000-0000-0000603d0055"
+					(reference "JP2")
+					(unit 1)
+				)
+			)
+		)
+	)
+	(symbol
 		(lib_id "power:GND")
 		(at 41.91 139.7 0)
@@
 					(unit 1)
 				)
+			)
+		)
+	)
+	(symbol
+		(lib_id "Jumper:SolderJumper_2_Bridged")
+		(at 95.25 113.03 90)
+		(unit 1)
+		(exclude_from_sim no)
+		(in_bom no)
+		(on_board yes)
+		(dnp no)
+		(property "Reference" "JP3"
+			(at 90.932 111.252 90)
+			(effects
+				(font
+					(size 1.27 1.27)
+				)
+			)
+		)
+		(property "Value" "CTS"
+			(at 91.186 113.03 90)
+			(effects
+				(font
+					(size 1.27 1.27)
+				)
+			)
+		)
+		(property "Footprint" "Jumper:SolderJumper-2_P1.3mm_Bridged_RoundedPad1.0x1.5mm"
+			(at 95.25 113.03 0)
+			(effects
+				(font
+					(size 1.27 1.27)
+				)
+				(hide yes)
+			)
+		)
+		(property "Datasheet" "~"
+			(at 95.25 113.03 0)
+			(effects
+				(font
+					(size 1.27 1.27)
+				)
+				(hide yes)
+			)
+		)
+		(property "Description" "Solder Jumper, 2-pole, closed/bridged"
+			(at 95.25 113.03 0)
+			(effects
+				(font
+					(size 1.27 1.27)
+				)
+				(hide yes)
+			)
+		)
+		(pin "2"
+		)
+		(pin "1"
+		)
+		(instances
+			(project "MCU-Link_MR"
+				(path "/5d025764-753a-4b80-8d3d-c9a8a22c9527/00000000-0000-0000-0000-0000603d0055"
+					(reference "JP3")
+					(unit 1)
+				)

Commit message: minor label placement
Parts:
- R26, R27: mouser# 652-CR0603-JW-100ELF -> 667-ERJ-2GEJ100X
- R28: mouser# 652-CR0603-JW-104ELF -> 791-MR04X104JTL
Changed lines of the file:
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@@
 			)
 		)
-		(property "mouser#" "652-CR0603-JW-104ELF"
+		(property "mouser#" "791-MR04X104JTL"
 			(at 67.31 39.37 0)
 			(effects
@@
 			)
 		)
-		(property "mouser#" "652-CR0603-JW-100ELF"
+		(property "mouser#" "667-ERJ-2GEJ100X "
 			(at 71.12 48.26 0)
 			(effects
@@
 			)
 		)
-		(property "mouser#" "652-CR0603-JW-100ELF"
+		(property "mouser#" "667-ERJ-2GEJ100X "
 			(at 71.12 86.36 0)
 			(effects

Commit message: updated BOM with new part numbers
Parts:
- C40, C41, C42, C43, C44, C45, C46, C47: value 100nF 6.3V -> 100nF 25V; mouser# 80-C0603C104K9R -> 963-MLAST105SB5104KF
- R25, R26, R27, R6: value 10R 5% 100mW -> 10R 1% 63mW; mouser# 667-ERJ-2GEJ100X -> 71-CRCW040210R0FKEDC
- R28, R5: value 100k 5% 100mW -> 100k 1% 63mW; mouser# 791-MR04X104JTL -> 71-CRCW0402100KFKEDC
Changed lines of the file:
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@@
 			)
 		)
-		(property "Value" "100k 5% 100mW"
+		(property "Value" "100k 1% 63mW"
 			(at 76.708 39.624 0)
 			(effects
@@
 			)
 		)
-		(property "mouser#" "791-MR04X104JTL"
+		(property "mouser#" "71-CRCW0402100KFKEDC"
 			(at 67.31 39.37 0)
 			(effects
@@
 			)
 		)
-		(property "Value" "100nF 6.3V"
+		(property "Value" "100nF 25V"
 			(at 43.18 30.226 90)
 			(effects
@@
 			)
 		)
-		(property "mouser#" "80-C0603C104K9R"
+		(property "mouser#" "963-MLAST105SB5104KF"
 			(at 46.99 34.29 0)
 			(effects
@@
 			)
 		)
-		(property "Value" "100nF 6.3V"
+		(property "Value" "100nF 25V"
 			(at 63.5 27.6606 90)
 			(effects
@@
 			)
 		)
-		(property "mouser#" "80-C0603C104K9R"
+		(property "mouser#" "963-MLAST105SB5104KF"
 			(at 63.5 31.75 0)
 			(effects
@@
 			)
 		)
-		(property "Value" "10R 5% 100mW"
+		(property "Value" "10R 1% 63mW"
 			(at 71.12 50.8 90)
 			(effects
@@
 			)
 		)
-		(property "mouser#" "667-ERJ-2GEJ100X "
+		(property "mouser#" "71-CRCW040210R0FKEDC"
 			(at 71.12 48.26 0)
 			(effects
@@
 			)
 		)
-		(property "Value" "100nF 6.3V"
+		(property "Value" "100nF 25V"
 			(at 43.18 68.326 90)
 			(effects
@@
 			)
 		)
-		(property "mouser#" "80-C0603C104K9R"
+		(property "mouser#" "963-MLAST105SB5104KF"
 			(at 46.99 72.39 0)
 			(effects
@@
 			)
 		)
-		(property "Value" "100nF 6.3V"
+		(property "Value" "100nF 25V"
 			(at 63.5 65.7606 90)
 			(effects
@@
 			)
 		)
-		(property "mouser#" "80-C0603C104K9R"
+		(property "mouser#" "963-MLAST105SB5104KF"
 			(at 63.5 69.85 0)
 			(effects
@@
 			)
 		)
-		(property "Value" "10R 5% 100mW"
+		(property "Value" "10R 1% 63mW"
 			(at 71.12 88.9 90)
 			(effects
@@
 			)
 		)
-		(property "mouser#" "667-ERJ-2GEJ100X "
+		(property "mouser#" "71-CRCW040210R0FKEDC"
 			(at 71.12 86.36 0)
 			(effects
@@
 			)
 		)
-		(property "Value" "100k 5% 100mW"
+		(property "Value" "100k 1% 63mW"
 			(at 84.328 138.684 0)
 			(effects
@@
 			)
 		)
-		(property "mouser#" "791-MR04X104JTL"
+		(property "mouser#" "71-CRCW0402100KFKEDC"
 			(at 74.93 138.43 0)
 			(effects
@@
 			)
 		)
-		(property "Value" "10R 5% 100mW"
+		(property "Value" "10R 1% 63mW"
 			(at 83.82 132.08 90)
 			(effects
@@
 			)
 		)
-		(property "mouser#" "667-ERJ-2GEJ100X "
+		(property "mouser#" "71-CRCW040210R0FKEDC"
 			(at 83.82 129.54 0)
 			(effects
@@
 			)
 		)
-		(property "Value" "10R 5% 100mW"
+		(property "Value" "10R 1% 63mW"
 			(at 69.85 176.53 90)
 			(effects
@@
 			)
 		)
-		(property "mouser#" "667-ERJ-2GEJ100X "
+		(property "mouser#" "71-CRCW040210R0FKEDC"
 			(at 69.85 173.99 0)
 			(effects
@@
 			)
 		)
-		(property "Value" "100nF 6.3V"
+		(property "Value" "100nF 25V"
 			(at 41.91 155.956 90)
 			(effects
@@
 			)
 		)
-		(property "mouser#" "80-C0603C104K9R"
+		(property "mouser#" "963-MLAST105SB5104KF"
 			(at 45.72 160.02 0)
 			(effects
@@
 			)
 		)
-		(property "Value" "100nF 6.3V"
+		(property "Value" "100nF 25V"
 			(at 62.23 153.3906 90)
 			(effects
@@
 			)
 		)
-		(property "mouser#" "80-C0603C104K9R"
+		(property "mouser#" "963-MLAST105SB5104KF"
 			(at 62.23 157.48 0)
 			(effects
@@
 			)
 		)
-		(property "Value" "100nF 6.3V"
+		(property "Value" "100nF 25V"
 			(at 43.18 111.506 90)
 			(effects
@@
 			)
 		)
-		(property "mouser#" "80-C0603C104K9R"
+		(property "mouser#" "963-MLAST105SB5104KF"
 			(at 46.99 115.57 0)
 			(effects
@@
 			)
 		)
-		(property "Value" "100nF 6.3V"
+		(property "Value" "100nF 25V"
 			(at 63.5 108.9406 90)
 			(effects
@@
 			)
 		)
-		(property "mouser#" "80-C0603C104K9R"
+		(property "mouser#" "963-MLAST105SB5104KF"
 			(at 63.5 113.03 0)
 			(effects
